File: tokypicokeeb.kicad_pcb (KiCad board)
At the start: 2 copper layers, 129 parts, among them SW1 SW_Push, U1 PicoW

Commit message: duplex trigger
Parts:
- moved D1 234.0 mm to (355.1, 120.6)
- moved D10 234.0 mm to (355.1, 150.7)
- moved D11 234.0 mm to (355.1, 154.1)
- moved D12 234.0 mm to (360.8, 120.6)
- moved D13 234.0 mm to (360.8, 123.9)
- moved D14 234.0 mm to (360.8, 127.3)
- moved D15 234.0 mm to (360.8, 130.6)
- moved D16 234.0 mm to (360.8, 134.0)
- moved D17 234.0 mm to (360.8, 137.3)
- moved D18 234.0 mm to (360.8, 140.7)
- moved D19 234.0 mm to (360.8, 144.0)
- moved D2 234.0 mm to (355.1, 123.9)
- moved D20 234.0 mm to (360.8, 147.4)
- moved D21 234.0 mm to (360.8, 150.7)
- moved D22 234.0 mm to (360.8, 154.1)
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