File: tokypicokeeb.kicad_pcb (KiCad board)
At the start: 2 copper layers, 129 parts, among them SW1 SW_Push, U1 PicoW

Commit message: 1/2 diodes
Parts:
- D1, D10, D11, D12, D13, D14, D15, D16, D17, D18, D19, D2, D20, D21, D22, D23, D24, D25, D26, D27, D28, D29, D3, D30, D31, D32, D33, D34, D35, D36, D37, D38, D39, D4, D40, D41, D42, D43, D44, D45, D46, D47, D48, D49, D5, D50, D51, D52, D53, D54, D55, D56, D57, D58, D59, D6, D60, D61, D62, D63, D7, D8, D9: footprint random-keyboard-parts:D_SOD-123-Pretty -> ScottoKeebs_Components:Diode_DO-35
- SHIFT1: footprint MX_Only:MXOnly-2.25U-ReversedStabilizers-NoLED -> MX_Only:MXOnly-2.25U-NoLED
- moved D10 441.3 mm to (-78.3, 67.7)
- moved D11 441.3 mm to (-78.3, 71.1)
- moved D12 441.3 mm to (-72.6, 37.6)
- moved D13 441.3 mm to (-72.6, 40.9)
- moved D20 441.3 mm to (-72.6, 64.4)
- moved D21 441.3 mm to (-72.6, 67.7)
- moved D22 441.3 mm to (-72.6, 71.1)
- moved D23 441.3 mm to (-66.8, 37.6)
- moved D24 441.3 mm to (-66.8, 40.9)
- moved D25 441.3 mm to (-66.8, 44.3)
- moved D26 441.3 mm to (-66.8, 47.6)
- moved D7 441.3 mm to (-78.3, 57.7)
- moved D8 441.3 mm to (-78.3, 61.0)
- moved D9 441.3 mm to (-78.3, 64.4)
- moved D39 441.3 mm to (-61.1, 54.3)
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
Commit message: finished the diodes placement
Parts:
- moved D13 252.6 mm to (175.4, -6.99), turned to -90 degrees
- moved D26 250.6 mm to (178.1, -5.40), turned to -90 degrees
- moved D52 247.2 mm to (183.7, -2.22), turned to -90 degrees
- moved D51 244.2 mm to (181.0, -3.81), turned to -90 degrees
- moved D61 242.4 mm to (186.5, -0.64), turned to -90 degrees
- moved D11 239.0 mm to (147.6, -6.99), turned to -90 degrees
- moved D12 238.2 mm to (161.5, -6.99), turned to -90 degrees
- moved D25 236.4 mm to (164.3, -5.40), turned to -90 degrees
- moved D50 232.2 mm to (169.9, -2.22), turned to -90 degrees
- moved D49 229.0 mm to (167.0, -3.81), turned to -90 degrees
- moved D60 228.1 mm to (172.6, -0.73), turned to -90 degrees
- moved D10 227.5 mm to (136.5, -6.99), turned to -90 degrees
- moved D24 222.1 mm to (150.4, -5.50), turned to -90 degrees
- moved D48 217.0 mm to (155.9, -2.32), turned to -90 degrees
- moved D47 214.0 mm to (153.2, -3.81), turned to -90 degrees
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
Commit message: finished ver. 1
Parts:
- removed R1: R_Small, Resistor_SMD:R_0805_2012Metric
- moved SW1 318.5 mm to (-12.4, 22.1)
- moved D11 15.7 mm to (163.1, -3.91)
- moved D13 15.7 mm to (190.8, -3.91)
- moved D22 15.7 mm to (140.8, -2.32)
- moved D24 15.7 mm to (165.8, -2.42)
- moved D26 15.7 mm to (193.6, -2.32)
- moved D43 15.7 mm to (143.6, -0.73)
- moved D47 15.7 mm to (168.6, -0.73)
- moved D48 15.7 mm to (171.3, 0.76)
- moved D51 15.7 mm to (196.4, -0.73)
- moved D52 15.7 mm to (199.1, 0.85)
- moved D21 15.7 mm to (127.0, -2.32)
- moved D41 15.7 mm to (129.7, -0.73)
- moved D42 15.7 mm to (132.6, 0.85)
- moved D57 15.7 mm to (135.3, 2.35)
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Connections:
- SW1 pad 1: GND -> Net-(SW1-Pad1)
- U1 pad 13: GND -> unconnected-(U1-GND-Pad13)
- U1 pad 18: GND -> unconnected-(U1-GND-Pad18)
- U1 pad 23: GND -> unconnected-(U1-GND-Pad23)
- U1 pad 28: GND -> unconnected-(U1-GND-Pad28)
- U1 pad 3: GND -> Net-(SW1-Pad1)
- U1 pad 36: +3.3V -> unconnected-(U1-3V3-Pad36)
- U1 pad 38: GND -> unconnected-(U1-GND-Pad38)
- U1 pad 40: +5V -> unconnected-(U1-VBUS-Pad40)
- U1 pad 42: GND -> unconnected-(U1-GND-Pad42)
- U1 pad 8: GND -> unconnected-(U1-GND-Pad8)
Routing:
- net Col 12: track 0.00 -> 357.6 mm
- net Col 11: track 0.00 -> 302.8 mm
- net Col 10: track 0.00 -> 288.0 mm
- net Col 8: track 0.00 -> 257.1 mm
- net Col 9: track 0.00 -> 253.2 mm
- net Col 6: track 0.00 -> 252.2 mm
- net Col 7: track 0.00 -> 240.8 mm
- net Row 0: track 0.00 -> 206.1 mm
- net Row 4: track 0.00 -> 203.4 mm
- net Row 1: track 0.00 -> 201.6 mm
- net Row 2: track 0.00 -> 199.9 mm
- net Row 3: track 0.00 -> 194.1 mm
- net Col 5: track 0.00 -> 191.8 mm
- net Col 4: track 0.00 -> 177.0 mm
- net Col 3: track 0.00 -> 159.3 mm
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- added copper zone on B.Cu, net (none)
- added copper zone on F.Cu, net (none)
Other:
- board outline added: 325.4 x 145.3 mm
